Commit message: Update: changed the make list to provide for the navigation goal and made modifications to chassis of robot

File: urdf/shane_bot.xacro (robot description, xacro)
@@ -25,8 +25,9 @@
 			/>
 		</inertial>
+		<!-- Main Chassis -->
 		<collision name="chassis_collision">
 			<origin xyz="0 0 0" rpy="0 0 0"/>
 			<geometry>
-				<box size="0.4 0.2 0.1"/>
+				<box size="0.2 0.2 0.1"/>
 			</geometry>
 		</collision>
@@ -34,10 +35,39 @@
 			<origin xyz="0 0 0" rpy="0 0 0"/>
 			<geometry>
-				<box size="0.4 0.2 0.1"/>
+				<box size="0.2 0.2 0.1"/>
 			</geometry>
 			<material name="blue"/>
 		</visual>
+		<!-- Front portion of chassis -->
+		<collision name="front_chassis_collision">
+			<origin xyz="0.2 0 0" rpy="0 0 0"/>
+			<geometry>
+				<box size="0.2 0.2 0.1"/>
+			</geometry>
+		</collision>
+		<visual name="front_chassis_visual">
+			<origin xyz="0.2 0 0" rpy="0 0 0"/>
+			<geometry>
+				<box size="0.2 0.2 0.1"/>
+			</geometry>
+			<material name="blue"/>
+		</visual>
+		<!-- Top portion of chassis -->
+		<collision name="top_chassis_collision">
+			<origin xyz="0 0 0.1" rpy="0 0 0"/>
+			<geometry>
+				<box size="0.2 0.2 0.1"/>
+			</geometry>
+		</collision>
+		<visual name="top_chassis_visual">
+			<origin xyz="0 0 0.1" rpy="0 0 0"/>
+			<geometry>
+				<box size="0.2 0.2 0.1"/>
+			</geometry>
+			<material name="blue"/>
+		</visual>
+		<!-- Caster at the back of robot -->
 		<collision name='back_caster_collision'>
-			<origin xyz="-0.15 0 -0.05" rpy="0 0 0"/>
+			<origin xyz="-0.05 0 -0.05" rpy="0 0 0"/>
 			<geometry>
 				<sphere radius="0.0499"/>
@@ -45,11 +75,12 @@
 		</collision>
 		<visual name="back_caster_visual">
-			<origin xyz="-0.15 0 -0.05" rpy="0 0 0"/>
+			<origin xyz="-0.05 0 -0.05" rpy="0 0 0"/>
 			<geometry>
 				<sphere radius="0.05"/>
 			</geometry>
 		</visual>
+		<!-- Caster at front of robot -->
 		<collision name='front_caster_visual'>
-			<origin xyz="0.15 0 -0.05" rpy="0 0 0"/>
+			<origin xyz="0.25 0 -0.05" rpy="0 0 0"/>
 			<geometry>
 				<sphere radius="0.0499"/>
@@ -57,5 +88,5 @@
 		</collision>
 		<visual name="front_caster_visual">
-			<origin xyz="0.15 0 -0.05" rpy="0 0 0"/>
+			<origin xyz="0.25 0 -0.05" rpy="0 0 0"/>
 			<geometry>
 				<sphere radius="0.05"/>
@@ -158,5 +189,5 @@
 	<!-- Joint connecting the camera to the chassis -->
 	<joint type="fixed" name="camera_joint">
-		<origin xyz="0.2 0 0" rpy="0 0 0"/>
+		<origin xyz="0.3 0 0" rpy="0 0 0"/>
 		<parent link="chassis"/>
 		<child link="camera"/>
@@ -188,5 +219,5 @@
 	<!-- Joint connecting the  -->
 	<joint type="fixed" name="hokuyo_joint">
-		<origin xyz="0.15 0 0.1" rpy="0 0 0"/>
+		<origin xyz="0 0 0.2" rpy="0 0 0"/>
 		<parent link="chassis"/>
 		<child link="hokuyo"/>
